File: hw2/PIC32_PCB/sch_design.brd (EAGLE design)
At the start: 100 x 100 mm, 23 parts, among them J1 USB-MB-H, J2 1x08, J3 1x08

Commit message: upload mouse control
Parts:
- moved C5 19.2 mm to (34.3, 62.2)
- moved J2 0.52 mm to (2.03, 57.0)
Changed lines of the file:
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@@
 <drawing>
 <settings>
-<setting alwaysvectorfont="no"/>
+<setting alwaysvectorfont="yes"/>
 <setting verticaltext="up"/>
 </settings>
@@
 </class>
 </classes>
-<designrules name="default">
+<designrules name="SeeedStudio_2layer_DRU_no_angle_20140221">
 <description language="de">&lt;b&gt;EAGLE Design Rules&lt;/b&gt;
 &lt;p&gt;
@@
 necessary adjustments and save your customized
 design rules under a new name.</description>
+<description language="zh">&lt;b&gt;Seeed Studio EAGLE Design Rules&lt;/b&gt;
+</description>
 <param name="layerSetup" value="(1*16)"/>
-<param name="mtCopper" value="0.035mm 0.035mm 0.035mm 0.035mm 0.035mm 0.035mm 0.035mm 0.035mm 0.035mm 0.035mm 0.035mm 0.035mm 0.035mm 0.035mm 0.035mm 0.035mm"/>
-<param name="mtIsolate" value="1.5mm 0.15mm 0.2mm 0.15mm 0.2mm 0.15mm 0.2mm 0.15mm 0.2mm 0.15mm 0.2mm 0.15mm 0.2mm 0.15mm 0.2mm"/>
+<param name="mtCopper" value="0.035mm 0.0175mm 0.035mm 0.035mm 0.035mm 0.035mm 0.035mm 0.035mm 0.035mm 0.035mm 0.035mm 0.035mm 0.035mm 0.035mm 0.0175mm 0.035mm"/>
+<param name="mtIsolate" value="1.5mm 1.1mm 0.2mm 0.15mm 0.2mm 0.15mm 0.2mm 0.15mm 0.2mm 0.15mm 0.2mm 0.15mm 0.2mm 0.15mm 0.2mm"/>
 <param name="mdWireWire" value="6mil"/>
 <param name="mdWirePad" value="6mil"/>
@@
 <param name="mdPadVia" value="6mil"/>
 <param name="mdViaVia" value="6mil"/>
-<param name="mdSmdPad" value="6mil"/>
-<param name="mdSmdVia" value="6mil"/>
-<param name="mdSmdSmd" value="6mil"/>
-<param name="mdViaViaSameLayer" value="6mil"/>
+<param name="mdSmdPad" value="0mil"/>
+<param name="mdSmdVia" value="0mil"/>
+<param name="mdSmdSmd" value="0mil"/>
+<param name="mdViaViaSameLayer" value="8mil"/>
 <param name="mnLayersViaInSmd" value="2"/>
-<param name="mdCopperDimension" value="40mil"/>
-<param name="mdDrill" value="6mil"/>
+<param name="mdCopperDimension" value="10mil"/>
+<param name="mdDrill" value="10mil"/>
 <param name="mdSmdStop" value="0mil"/>
 <param name="msWidth" value="6mil"/>
-<param name="msDrill" value="0.35mm"/>
-<param name="msMicroVia" value="9.99mm"/>
+<param name="msDrill" value="12mil"/>
+<param name="msMicroVia" value="12mil"/>
 <param name="msBlindViaRatio" value="0.5"/>
 <param name="rvPadTop" value="0.25"/>
@@
 <param name="rlMinPadBottom" value="10mil"/>
 <param name="rlMaxPadBottom" value="20mil"/>
-<param name="rlMinViaOuter" value="8mil"/>
+<param name="rlMinViaOuter" value="6mil"/>
 <param name="rlMaxViaOuter" value="20mil"/>
-<param name="rlMinViaInner" value="8mil"/>
+<param name="rlMinViaInner" value="6mil"/>
 <param name="rlMaxViaInner" value="20mil"/>
 <param name="rlMinMicroViaOuter" value="4mil"/>
@@
 <param name="psTop" value="-1"/>
 <param name="psBottom" value="-1"/>
-<param name="psFirst" value="-1"/>
+<param name="psFirst" value="0"/>
 <param name="psElongationLong" value="100"/>
 <param name="psElongationOffset" value="100"/>
 <param name="mvStopFrame" value="1"/>
 <param name="mvCreamFrame" value="0"/>
-<param name="mlMinStopFrame" value="4mil"/>
-<param name="mlMaxStopFrame" value="4mil"/>
+<param name="mlMinStopFrame" value="2mil"/>
+<param name="mlMaxStopFrame" value="2mil"/>
 <param name="mlMinCreamFrame" value="0mil"/>
 <param name="mlMaxCreamFrame" value="0mil"/>
-<param name="mlViaStopLimit" value="0mil"/>
+<param name="mlViaStopLimit" value="100mil"/>
 <param name="srRoundness" value="0"/>
 <param name="srMinRoundness" value="0mil"/>
@@
 <param name="checkAngle" value="0"/>
 <param name="checkFont" value="1"/>
-<param name="checkRestrict" value="1"/>
+<param name="checkRestrict" value="0"/>
 <param name="checkStop" value="0"/>
 <param name="checkValues" value="0"/>
@@
 <attribute name="VALUE" x="18.034" y="50.546" size="1.27" layer="27" ratio="10"/>
 </element>
-<element name="C5" library="rcl" library_urn="urn:adsk.eagle:library:334" package="B45181B" package3d_urn="urn:adsk.eagle:package:23320/1" value="10uF" x="36.83" y="43.18" smashed="yes" rot="R270">
-<attribute name="NAME" x="39.624" y="46.101" size="1.27" layer="25" ratio="10" rot="R270"/>
-<attribute name="SPICEPREFIX" value="C" x="21.59" y="8.89" size="1.778" layer="27" rot="R270" display="off"/>
-<attribute name="VALUE" x="35.179" y="38.989" size="1.27" layer="27" ratio="10" rot="R270"/>
+<element name="C5" library="rcl" library_urn="urn:adsk.eagle:library:334" package="B45181B" package3d_urn="urn:adsk.eagle:package:23320/1" value="10uF" x="34.29" y="62.23" smashed="yes" rot="R270">
+<attribute name="NAME" x="37.084" y="65.151" size="1.27" layer="25" ratio="10" rot="R270"/>
+<attribute name="SPICEPREFIX" value="C" x="19.05" y="27.94" size="1.778" layer="27" rot="R270" display="off"/>
+<attribute name="VALUE" x="32.639" y="58.039" size="1.27" layer="27" ratio="10" rot="R270"/>
 </element>
 <element name="C6" library="rcl" library_urn="urn:adsk.eagle:library:334" package="B45181B" package3d_urn="urn:adsk.eagle:package:23320/1" value="10uF" x="13.97" y="82.55" smashed="yes" rot="R180">
@@
 <attribute name="NAME" x="11.822" y="94.845" size="1.27" layer="25" rot="R90"/>
 </element>
-<element name="J2" library="pic32_lib" package="1X08" value="1x08" x="2.54" y="57.15" smashed="yes" rot="R270">
-<attribute name="NAME" x="3.937" y="58.42" size="0.6096" layer="25" font="vector" ratio="20" rot="R270"/>
-<attribute name="PROD_ID" value="CONN-08438" x="-46.99" y="5.08" size="1.778" layer="27" rot="R270" display="off"/>
-<attribute name="VALUE" x="0.508" y="58.42" size="0.6096" layer="27" font="vector" ratio="20" rot="R270"/>
+<element name="J2" library="pic32_lib" package="1X08" value="1x08" x="2.032" y="57.023" smashed="yes" rot="R270">
+<attribute name="NAME" x="3.429" y="58.293" size="0.6096" layer="25" font="vector" ratio="20" rot="R270"/>
+<attribute name="PROD_ID" value="CONN-08438" x="-47.498" y="4.953" size="1.778" layer="27" rot="R270" display="off"/>
+<attribute name="VALUE" x="0" y="58.293" size="0.6096" layer="27" font="vector" ratio="20" rot="R270"/>
 </element>
 <element name="J3" library="pic32_lib" package="1X08" value="1x08" x="97.917" y="58.42" smashed="yes" rot="R270">
@@
 <vertex x="-2.54" y="102.87"/>
 </polygon>
+<polygon width="0.1524" layer="16" isolate="0.3048">
+<vertex x="0.254" y="99.695"/>
+<vertex x="99.695" y="99.695"/>
+<vertex x="99.695" y="0.127"/>
+<vertex x="0.127" y="0.127"/>
+<vertex x="0" y="0"/>
+<vertex x="0" y="99.314"/>
+<vertex x="0.254" y="99.568"/>
+</polygon>
 <wire x1="49.53" y1="57.87" x2="55.33" y2="52.87" width="0" layer="19" extent="1-1"/>
 <wire x1="43.73" y1="52.07" x2="49.53" y2="57.87" width="0" layer="19" extent="1-1"/>
 <wire x1="48.73" y1="46.27" x2="43.73" y2="52.07" width="0" layer="19" extent="1-1"/>
-<wire x1="45.72" y1="31.75" x2="48.73" y2="46.27" width="0" layer="19" extent="1-1"/>
+<wire x1="34.29" y1="59.69" x2="43.73" y2="52.07" width="0" layer="19" extent="1-1"/>
 </signal>
 <signal name="N$1">
@@
 <wire x1="30.48" y1="68.58" x2="19.685" y2="69.85" width="0" layer="19" extent="1-1"/>
 <wire x1="47.13" y1="57.87" x2="30.48" y2="68.58" width="0" layer="19" extent="1-1"/>
-<wire x1="2.54" y1="54.61" x2="19.685" y2="69.85" width="0" layer="19" extent="1-1"/>
+<wire x1="2.032" y1="54.483" x2="19.685" y2="69.85" width="0" layer="19" extent="1-1"/>
 </signal>
 <signal name="+3V3">
@@
 <wire x1="69.85" y1="15.24" x2="66.04" y2="27.94" width="0" layer="19" extent="1-1"/>
 <wire x1="53.34" y1="15.24" x2="69.85" y2="15.24" width="0" layer="19" extent="1-1"/>
-<wire x1="48.26" y1="31.75" x2="66.04" y2="27.94" width="0" layer="19" extent="1-1"/>
+<wire x1="48.26" y1="31.75" x2="53.34" y2="15.24" width="0" layer="19" extent="1-1"/>
 <wire x1="49.53" y1="46.27" x2="48.26" y2="31.75" width="0" layer="19" extent="1-1"/>
 <wire x1="43.73" y1="48.87" x2="49.53" y2="46.27" width="0" layer="19" extent="1-1"/>
@@
 <contactref element="J2" pad="4"/>
 <contactref element="U$8" pad="44"/>
-<wire x1="2.54" y1="49.53" x2="45.53" y2="57.87" width="0" layer="19" extent="1-1"/>
+<wire x1="2.032" y1="49.403" x2="45.53" y2="57.87" width="0" layer="19" extent="1-1"/>
 </signal>
 <signal name="B7">
 <contactref element="J2" pad="3"/>
 <contactref element="U$8" pad="43"/>
-<wire x1="2.54" y1="52.07" x2="46.33" y2="57.87" width="0" layer="19" extent="1-1"/>
+<wire x1="2.032" y1="51.943" x2="46.33" y2="57.87" width="0" layer="19" extent="1-1"/>
 </signal>
 <signal name="B9">
 <contactref element="J2" pad="5"/>
 <contactref element="U$8" pad="1"/>
-<wire x1="2.54" y1="46.99" x2="43.73" y2="56.07" width="0" layer="19" extent="1-1"/>
+<wire x1="2.032" y1="46.863" x2="43.73" y2="56.07" width="0" layer="19" extent="1-1"/>
 </signal>
 <signal name="D+">
 <contactref element="J1" pad="D+"/>
 <contactref element="U$8" pad="8"/>
-<wire x1="9.672" y1="93.345" x2="43.73" y2="50.47" width="0" layer="19" extent="1-1"/>
+<wire x1="43.73" y1="50.47" x2="9.672" y2="93.345" width="0" layer="19" extent="1-1"/>
 </signal>
 <signal name="D-">
@@
 <contactref element="J2" pad="6"/>
 <contactref element="U$8" pad="11"/>
-<wire x1="2.54" y1="44.45" x2="43.73" y2="48.07" width="0" layer="19" extent="1-1"/>
+<wire x1="2.032" y1="44.323" x2="43.73" y2="48.07" width="0" layer="19" extent="1-1"/>
 </signal>
 <signal name="B14">
 <contactref element="J2" pad="7"/>
 <contactref element="U$8" pad="14"/>
-<wire x1="2.54" y1="41.91" x2="47.13" y2="46.27" width="0" layer="19" extent="1-1"/>
+<wire x1="2.032" y1="41.783" x2="47.13" y2="46.27" width="0" layer="19" extent="1-1"/>
 </signal>
 <signal name="B15">
 <contactref element="J2" pad="8"/>
 <contactref element="U$8" pad="15"/>
-<wire x1="2.54" y1="39.37" x2="47.93" y2="46.27" width="0" layer="19" extent="1-1"/>
+<wire x1="2.032" y1="39.243" x2="47.93" y2="46.27" width="0" layer="19" extent="1-1"/>
 </signal>
 <signal name="N$2">
 <contactref element="U$8" pad="7"/>
 <contactref element="C5" pad="+"/>
-<wire x1="36.83" y1="45.72" x2="43.73" y2="51.27" width="0" layer="19" extent="1-1"/>
+<wire x1="43.73" y1="51.27" x2="34.29" y2="64.77" width="0" layer="19" extent="1-1"/>
 </signal>
 <signal name="OSC2">
